File: Poncho_Alarma/Salidas.sch (KiCad schematic (older format))
At the start: 12 parts

Commit message: Esquematico Terminado
Parts:
- added J2: Salidas, symbol Connector_Generic:Conn_01x06
- K1, K2: renamed from K?; symbol PonchoPLC:RELAY_C -> Poncho_Alarma-rescue:RELAY_C-PonchoPLC
- gave numbers to parts that had none: 10
Connections:
- net at K2.1: now also J2.6 (Pin_6)
- net at K2.3: now also J2.5 (Pin_5)
- net at K2.4: now also J2.4 (Pin_4)
- net at K1.1: now also J2.3 (Pin_3)
- net at K1.3: now also J2.2 (Pin_2)
- net at K1.4: now also J2.1 (Pin_1)
Changed lines of the file:
@@
 encoding utf-8
 Sheet 2 3
-Title ""
-Date ""
-Rev ""
-Comp ""
-Comment1 ""
-Comment2 ""
+Title "Salidas"
+Date "2018-10-27"
+Rev "1.0"
+Comp "Proyecto CIAA - COMPUTADORA INDUSTRIAL ABIERTA ARGENTINA"
+Comment1 "https://github.com/turcoale/CESE18_PCB_Amid_Ale.git"
+Comment2 "Autor: Amid Ale"
 Comment3 ""
-Comment4 ""
+Comment4 "CÓDIGO PONCHO: ALARMA"
 $EndDescr
 Wire Wire Line
 	6300 3950 6300 4300
 $Comp
-L PonchoPLC:RELAY_C K?
+L Poncho_Alarma-rescue:RELAY_C-PonchoPLC K2
 U 1 1 5BD28B64
 P 6450 3750
-F 0 "K?" V 6503 3559 60  0000 R CNN
+F 0 "K2" V 6503 3559 60  0000 R CNN
 F 1 "RELAY_C" V 6397 3559 60  0000 R CNN
 F 2 "" H 6450 3750 60  0000 C CNN
@@
 $EndComp
 $Comp
-L Transistor_FET:2N7002 Q?
+L Transistor_FET:2N7002 Q2
 U 1 1 5BD28B6B
 P 5600 4500
-F 0 "Q?" H 5805 4546 50  0000 L CNN
+F 0 "Q2" H 5805 4546 50  0000 L CNN
 F 1 "2N7002" H 5805 4455 50  0000 L CNN
 F 2 "Package_TO_SOT_SMD:SOT-23" H 5800 4425 50  0001 L CIN
@@
 	5050 4500 5400 4500
 $Comp
-L power:GND #PWR?
+L power:GND #PWR0106
 U 1 1 5BD28B74
 P 5050 5000
-F 0 "#PWR?" H 5050 4750 50  0001 C CNN
+F 0 "#PWR0106" H 5050 4750 50  0001 C CNN
 F 1 "GND" H 5055 4827 50  0000 C CNN
 F 2 "" H 5050 5000 50  0001 C CNN
@@
 $EndComp
 $Comp
-L power:GND #PWR?
+L power:GND #PWR0107
 U 1 1 5BD28B7A
 P 5700 4850
-F 0 "#PWR?" H 5700 4600 50  0001 C CNN
+F 0 "#PWR0107" H 5700 4600 50  0001 C CNN
 F 1 "GND" H 5705 4677 50  0000 C CNN
 F 2 "" H 5700 4850 50  0001 C CNN
@@
 	5700 4850 5700 4700
 $Comp
-L Diode:LL4148 D?
+L Diode:LL4148 D4
 U 1 1 5BD28B81
 P 5700 3850
-F 0 "D?" V 5654 3929 50  0000 L CNN
+F 0 "D4" V 5654 3929 50  0000 L CNN
 F 1 "LL4148" V 5745 3929 50  0000 L CNN
 F 2 "Diode_SMD:D_MiniMELF" H 5700 3675 50  0001 C CNN
@@
 $EndComp
 $Comp
-L Device:LED_Small_ALT D?
+L Device:LED_Small_ALT D2
 U 1 1 5BD28B88
 P 5300 3700
-F 0 "D?" V 5346 3632 50  0000 R CNN
+F 0 "D2" V 5346 3632 50  0000 R CNN
 F 1 "LED_Rojo" V 5200 3700 50  0000 R CNN
 F 2 "" V 5300 3700 50  0001 C CNN
@@
 $EndComp
 $Comp
-L Device:R_Small R?
+L Device:R_Small R3
 U 1 1 5BD28B8F
 P 5050 4750
-F 0 "R?" H 5109 4796 50  0000 L CNN
+F 0 "R3" H 5109 4796 50  0000 L CNN
 F 1 "100k" H 5109 4705 50  0000 L CNN
 F 2 "" H 5050 4750 50  0001 C CNN
@@
 	5050 4850 5050 5000
 $Comp
-L Device:R_Small R?
+L Device:R_Small R5
 U 1 1 5BD28B97
 P 5300 4050
-F 0 "R?" H 5359 4096 50  0000 L CNN
+F 0 "R5" H 5359 4096 50  0000 L CNN
 F 1 "330" H 5359 4005 50  0000 L CNN
 F 2 "" H 5300 4050 50  0001 C CNN
@@
 	5700 3550 6300 3550
 $Comp
-L power:+5V #PWR?
+L power:+5V #PWR0108
 U 1 1 5BD28BA4
 P 5700 3450
-F 0 "#PWR?" H 5700 3300 50  0001 C CNN
+F 0 "#PWR0108" H 5700 3300 50  0001 C CNN
 F 1 "+5V" H 5715 3623 50  0000 C CNN
 F 2 "" H 5700 3450 50  0001 C CNN
@@
 	6300 1850 6300 2200
 $Comp
-L PonchoPLC:RELAY_C K?
+L Poncho_Alarma-rescue:RELAY_C-PonchoPLC K1
 U 1 1 5BD28BB1
 P 6450 1650
-F 0 "K?" V 6503 1459 60  0000 R CNN
+F 0 "K1" V 6503 1459 60  0000 R CNN
 F 1 "RELAY_C" V 6397 1459 60  0000 R CNN
 F 2 "" H 6450 1650 60  0000 C CNN
@@
 $EndComp
 $Comp
-L Transistor_FET:2N7002 Q?
+L Transistor_FET:2N7002 Q1
 U 1 1 5BD28BB8
 P 5600 2400
-F 0 "Q?" H 5805 2446 50  0000 L CNN
+F 0 "Q1" H 5805 2446 50  0000 L CNN
 F 1 "2N7002" H 5805 2355 50  0000 L CNN
 F 2 "Package_TO_SOT_SMD:SOT-23" H 5800 2325 50  0001 L CIN
@@
 	5050 2400 5400 2400
 $Comp
-L power:GND #PWR?
+L power:GND #PWR0109
 U 1 1 5BD28BC1
 P 5050 2900
-F 0 "#PWR?" H 5050 2650 50  0001 C CNN
+F 0 "#PWR0109" H 5050 2650 50  0001 C CNN
 F 1 "GND" H 5055 2727 50  0000 C CNN
 F 2 "" H 5050 2900 50  0001 C CNN
@@
 $EndComp
 $Comp
-L power:GND #PWR?
+L power:GND #PWR0110
 U 1 1 5BD28BC7
 P 5700 2750
-F 0 "#PWR?" H 5700 2500 50  0001 C CNN
+F 0 "#PWR0110" H 5700 2500 50  0001 C CNN
 F 1 "GND" H 5705 2577 50  0000 C CNN
 F 2 "" H 5700 2750 50  0001 C CNN
@@
 	5700 2750 5700 2600
 $Comp
-L Diode:LL4148 D?
+L Diode:LL4148 D3
 U 1 1 5BD28BCE
 P 5700 1750
-F 0 "D?" V 5654 1829 50  0000 L CNN
+F 0 "D3" V 5654 1829 50  0000 L CNN
 F 1 "LL4148" V 5745 1829 50  0000 L CNN
 F 2 "Diode_SMD:D_MiniMELF" H 5700 1575 50  0001 C CNN
@@
 $EndComp
 $Comp
-L Device:LED_Small_ALT D?
+L Device:LED_Small_ALT D1
 U 1 1 5BD28BD5
 P 5300 1600
-F 0 "D?" V 5346 1532 50  0000 R CNN
+F 0 "D1" V 5346 1532 50  0000 R CNN
 F 1 "LED_Rojo" V 5200 1600 50  0000 R CNN
 F 2 "" V 5300 1600 50  0001 C CNN
@@
 $EndComp
 $Comp
-L Device:R_Small R?
+L Device:R_Small R2
 U 1 1 5BD28BDC
 P 5050 2650
-F 0 "R?" H 5109 2696 50  0000 L CNN
+F 0 "R2" H 5109 2696 50  0000 L CNN
 F 1 "100k" H 5109 2605 50  0000 L CNN
 F 2 "" H 5050 2650 50  0001 C CNN
@@
 	5050 2750 5050 2900
 $Comp
-L Device:R_Small R?
+L Device:R_Small R4
 U 1 1 5BD28BE4
 P 5300 1950
-F 0 "R?" H 5359 1996 50  0000 L CNN
+F 0 "R4" H 5359 1996 50  0000 L CNN
 F 1 "330" H 5359 1905 50  0000 L CNN
 F 2 "" H 5300 1950 50  0001 C CNN
@@
 	5700 1450 6300 1450
 $Comp
-L power:+5V #PWR?
+L power:+5V #PWR0111
 U 1 1 5BD28BF1
 P 5700 1350
-F 0 "#PWR?" H 5700 1200 50  0001 C CNN
+F 0 "#PWR0111" H 5700 1200 50  0001 C CNN
 F 1 "+5V" H 5715 1523 50  0000 C CNN
 F 2 "" H 5700 1350 50  0001 C CNN
@@
 Text HLabel 5300 3550 0    50   Input ~ 0
 Out_2
+$Comp
+L Connector_Generic:Conn_01x06 J2
+U 1 1 5BDADE5B
+P 7550 2950
+F 0 "J2" H 7630 2942 50  0000 L CNN
+F 1 "Salidas" H 7630 2851 50  0000 L CNN
+F 2 "" H 7550 2950 50  0001 C CNN
+F 3 "~" H 7550 2950 50  0001 C CNN
+	1    7550 2950
+	1    0    0    -1
+$EndComp
+Wire Wire Line
+	6550 1850 6550 2950
+Wire Wire Line
+	6550 2950 7350 2950
+Wire Wire Line
+	6600 1450 6950 1450
+Wire Wire Line
+	6950 1450 6950 2850
+Wire Wire Line
+	6950 2850 7350 2850
+Wire Wire Line
+	6500 1450 6500 1300
+Wire Wire Line
+	6500 1300 7350 1300
+Wire Wire Line
+	7350 1300 7350 2750
+Wire Wire Line
+	6500 3550 6500 3050
+Wire Wire Line
+	6500 3050 7350 3050
+Wire Wire Line
+	6600 3550 6600 3150
+Wire Wire Line
+	6600 3150 7350 3150
+Wire Wire Line
+	6550 3950 7350 3950
+Wire Wire Line
+	7350 3950 7350 3250
 $EndSCHEMATC

Commit message: asociando componentes
Parts:
- D1, D2: footprint (none) -> LED_SMD:LED_0603_1608Metric_Pad1.05x0.95mm_HandSolder
- J2: footprint (none) -> TerminalBlock:TerminalBlock_bornier-6_P5.08mm
- K1, K2: footprint (none) -> Poncho-PLC:Relay_C
- Q1, Q2: footprint Package_TO_SOT_SMD:SOT-23 -> Poncho-PLC:SOT23
- R2, R3, R4, R5: footprint (none) -> Resistor_SMD:R_0603_1608Metric_Pad1.05x0.95mm_HandSolder
Changed lines of the file:
@@
 F 0 "K2" V 6503 3559 60  0000 R CNN
 F 1 "RELAY_C" V 6397 3559 60  0000 R CNN
-F 2 "" H 6450 3750 60  0000 C CNN
+F 2 "Poncho-PLC:Relay_C" H 6450 3750 60  0001 C CNN
 F 3 "" H 6450 3750 60  0000 C CNN
 	1    6450 3750
@@
 F 0 "Q2" H 5805 4546 50  0000 L CNN
 F 1 "2N7002" H 5805 4455 50  0000 L CNN
-F 2 "Package_TO_SOT_SMD:SOT-23" H 5800 4425 50  0001 L CIN
+F 2 "Poncho-PLC:SOT23" H 5800 4425 50  0001 L CIN
 F 3 "https://www.fairchildsemi.com/datasheets/2N/2N7002.pdf" H 5600 4500 50  0001 L CNN
 	1    5600 4500
@@
 F 0 "D2" V 5346 3632 50  0000 R CNN
 F 1 "LED_Rojo" V 5200 3700 50  0000 R CNN
-F 2 "" V 5300 3700 50  0001 C CNN
+F 2 "LED_SMD:LED_0603_1608Metric_Pad1.05x0.95mm_HandSolder" V 5300 3700 50  0001 C CNN
 F 3 "~" V 5300 3700 50  0001 C CNN
 	1    5300 3700
@@
 F 0 "R3" H 5109 4796 50  0000 L CNN
 F 1 "100k" H 5109 4705 50  0000 L CNN
-F 2 "" H 5050 4750 50  0001 C CNN
+F 2 "Resistor_SMD:R_0603_1608Metric_Pad1.05x0.95mm_HandSolder" H 5050 4750 50  0001 C CNN
 F 3 "~" H 5050 4750 50  0001 C CNN
 	1    5050 4750
@@
 F 0 "R5" H 5359 4096 50  0000 L CNN
 F 1 "330" H 5359 4005 50  0000 L CNN
-F 2 "" H 5300 4050 50  0001 C CNN
+F 2 "Resistor_SMD:R_0603_1608Metric_Pad1.05x0.95mm_HandSolder" H 5300 4050 50  0001 C CNN
 F 3 "~" H 5300 4050 50  0001 C CNN
 	1    5300 4050
@@
 F 0 "K1" V 6503 1459 60  0000 R CNN
 F 1 "RELAY_C" V 6397 1459 60  0000 R CNN
-F 2 "" H 6450 1650 60  0000 C CNN
+F 2 "Poncho-PLC:Relay_C" H 6450 1650 60  0001 C CNN
 F 3 "" H 6450 1650 60  0000 C CNN
 	1    6450 1650
@@
 F 0 "Q1" H 5805 2446 50  0000 L CNN
 F 1 "2N7002" H 5805 2355 50  0000 L CNN
-F 2 "Package_TO_SOT_SMD:SOT-23" H 5800 2325 50  0001 L CIN
+F 2 "Poncho-PLC:SOT23" H 5800 2325 50  0001 L CIN
 F 3 "https://www.fairchildsemi.com/datasheets/2N/2N7002.pdf" H 5600 2400 50  0001 L CNN
 	1    5600 2400
@@
 F 0 "D1" V 5346 1532 50  0000 R CNN
 F 1 "LED_Rojo" V 5200 1600 50  0000 R CNN
-F 2 "" V 5300 1600 50  0001 C CNN
+F 2 "LED_SMD:LED_0603_1608Metric_Pad1.05x0.95mm_HandSolder" V 5300 1600 50  0001 C CNN
 F 3 "~" V 5300 1600 50  0001 C CNN
 	1    5300 1600
@@
 F 0 "R2" H 5109 2696 50  0000 L CNN
 F 1 "100k" H 5109 2605 50  0000 L CNN
-F 2 "" H 5050 2650 50  0001 C CNN
+F 2 "Resistor_SMD:R_0603_1608Metric_Pad1.05x0.95mm_HandSolder" H 5050 2650 50  0001 C CNN
 F 3 "~" H 5050 2650 50  0001 C CNN
 	1    5050 2650
@@
 F 0 "R4" H 5359 1996 50  0000 L CNN
 F 1 "330" H 5359 1905 50  0000 L CNN
-F 2 "" H 5300 1950 50  0001 C CNN
+F 2 "Resistor_SMD:R_0603_1608Metric_Pad1.05x0.95mm_HandSolder" H 5300 1950 50  0001 C CNN
 F 3 "~" H 5300 1950 50  0001 C CNN
 	1    5300 1950
@@
 F 0 "J2" H 7630 2942 50  0000 L CNN
 F 1 "Salidas" H 7630 2851 50  0000 L CNN
-F 2 "" H 7550 2950 50  0001 C CNN
+F 2 "TerminalBlock:TerminalBlock_bornier-6_P5.08mm" H 7550 2950 50  0001 C CNN
 F 3 "~" H 7550 2950 50  0001 C CNN
 	1    7550 2950

Commit message: arreglado lo de la libreria
Parts:
- D1, D2: footprint LED_SMD:LED_0603_1608Metric_Pad1.05x0.95mm_HandSolder -> LED_THT:LED_D3.0mm
- D3, D4: footprint Diode_SMD:D_MiniMELF -> Diode_THT:D_DO-201AD_P12.70mm_Horizontal
- R2, R3, R4, R5: footprint Resistor_SMD:R_0603_1608Metric_Pad1.05x0.95mm_HandSolder -> Resistor_THT:R_Axial_DIN0204_L3.6mm_D1.6mm_P5.08mm_Horizontal
Changed lines of the file:
@@
 F 0 "D4" V 5654 3929 50  0000 L CNN
 F 1 "LL4148" V 5745 3929 50  0000 L CNN
-F 2 "Diode_SMD:D_MiniMELF" H 5700 3675 50  0001 C CNN
+F 2 "Diode_THT:D_DO-201AD_P12.70mm_Horizontal" H 5700 3675 50  0001 C CNN
 F 3 "http://www.vishay.com/docs/85557/ll4148.pdf" H 5700 3850 50  0001 C CNN
 	1    5700 3850
@@
 F 0 "D2" V 5346 3632 50  0000 R CNN
 F 1 "LED_Rojo" V 5200 3700 50  0000 R CNN
-F 2 "LED_SMD:LED_0603_1608Metric_Pad1.05x0.95mm_HandSolder" V 5300 3700 50  0001 C CNN
+F 2 "LED_THT:LED_D3.0mm" V 5300 3700 50  0001 C CNN
 F 3 "~" V 5300 3700 50  0001 C CNN
 	1    5300 3700
@@
 F 0 "R3" H 5109 4796 50  0000 L CNN
 F 1 "100k" H 5109 4705 50  0000 L CNN
-F 2 "Resistor_SMD:R_0603_1608Metric_Pad1.05x0.95mm_HandSolder" H 5050 4750 50  0001 C CNN
+F 2 "Resistor_THT:R_Axial_DIN0204_L3.6mm_D1.6mm_P5.08mm_Horizontal" H 5050 4750 50  0001 C CNN
 F 3 "~" H 5050 4750 50  0001 C CNN
 	1    5050 4750
@@
 F 0 "R5" H 5359 4096 50  0000 L CNN
 F 1 "330" H 5359 4005 50  0000 L CNN
-F 2 "Resistor_SMD:R_0603_1608Metric_Pad1.05x0.95mm_HandSolder" H 5300 4050 50  0001 C CNN
+F 2 "Resistor_THT:R_Axial_DIN0204_L3.6mm_D1.6mm_P5.08mm_Horizontal" H 5300 4050 50  0001 C CNN
 F 3 "~" H 5300 4050 50  0001 C CNN
 	1    5300 4050
@@
 F 0 "D3" V 5654 1829 50  0000 L CNN
 F 1 "LL4148" V 5745 1829 50  0000 L CNN
-F 2 "Diode_SMD:D_MiniMELF" H 5700 1575 50  0001 C CNN
+F 2 "Diode_THT:D_DO-201AD_P12.70mm_Horizontal" H 5700 1575 50  0001 C CNN
 F 3 "http://www.vishay.com/docs/85557/ll4148.pdf" H 5700 1750 50  0001 C CNN
 	1    5700 1750
@@
 F 0 "D1" V 5346 1532 50  0000 R CNN
 F 1 "LED_Rojo" V 5200 1600 50  0000 R CNN
-F 2 "LED_SMD:LED_0603_1608Metric_Pad1.05x0.95mm_HandSolder" V 5300 1600 50  0001 C CNN
+F 2 "LED_THT:LED_D3.0mm" V 5300 1600 50  0001 C CNN
 F 3 "~" V 5300 1600 50  0001 C CNN
 	1    5300 1600
@@
 F 0 "R2" H 5109 2696 50  0000 L CNN
 F 1 "100k" H 5109 2605 50  0000 L CNN
-F 2 "Resistor_SMD:R_0603_1608Metric_Pad1.05x0.95mm_HandSolder" H 5050 2650 50  0001 C CNN
+F 2 "Resistor_THT:R_Axial_DIN0204_L3.6mm_D1.6mm_P5.08mm_Horizontal" H 5050 2650 50  0001 C CNN
 F 3 "~" H 5050 2650 50  0001 C CNN
 	1    5050 2650
@@
 F 0 "R4" H 5359 1996 50  0000 L CNN
 F 1 "330" H 5359 1905 50  0000 L CNN
-F 2 "Resistor_SMD:R_0603_1608Metric_Pad1.05x0.95mm_HandSolder" H 5300 1950 50  0001 C CNN
+F 2 "Resistor_THT:R_Axial_DIN0204_L3.6mm_D1.6mm_P5.08mm_Horizontal" H 5300 1950 50  0001 C CNN
 F 3 "~" H 5300 1950 50  0001 C CNN
 	1    5300 1950

Commit message: Posicionado terminado
Connections:
- net K2_C: now reaches J2.6 (Pin_6), K2.1
- net K2_NA: now reaches J2.5 (Pin_5), K2.3
- net K2_NC: now reaches J2.4 (Pin_4), K2.4
- net K1_C: now reaches J2.3 (Pin_3), K1.1
- net K1_NA: now reaches J2.2 (Pin_2), K1.3
- net K1_NC: now reaches J2.1 (Pin_1), K1.4
Changed lines of the file:
@@
 Wire Wire Line
 	7350 3950 7350 3250
+Text Label 6950 2950 0    50   ~ 0
+K1_C
+Text Label 6950 2850 0    50   ~ 0
+K1_NA
+Text Label 7350 2550 0    50   ~ 0
+K1_NC
+Text Label 7150 3950 0    50   ~ 0
+K2_C
+Text Label 7150 3150 0    50   ~ 0
+K2_NA
+Text Label 7150 3050 0    50   ~ 0
+K2_NC
 $EndSCHEMATC

Commit message: Correcciónes
Connections:
- net Out_2: now reaches Q2.1 (G), R3.1
Changed lines of the file:
@@
 Comp "Proyecto CIAA - COMPUTADORA INDUSTRIAL ABIERTA ARGENTINA"
 Comment1 "https://github.com/turcoale/CESE18_PCB_Amid_Ale.git"
-Comment2 "Autor: Amid Ale"
-Comment3 ""
+Comment2 "Basado en diseños anteriores: Mariano Bustos - Jorge Osio - Diego Brengi"
+Comment3 "Autor: Amid Ale"
 Comment4 "CÓDIGO PONCHO: ALARMA"
 $EndDescr
@@
 $EndComp
 $Comp
-L power:GND #PWR0107
-U 1 1 5BD28B7A
-P 5700 4850
-F 0 "#PWR0107" H 5700 4600 50  0001 C CNN
-F 1 "GND" H 5705 4677 50  0000 C CNN
-F 2 "" H 5700 4850 50  0001 C CNN
-F 3 "" H 5700 4850 50  0001 C CNN
-	1    5700 4850
-	1    0    0    -1
-$EndComp
-Wire Wire Line
-	5700 4850 5700 4700
-$Comp
 L Diode:LL4148 D4
 U 1 1 5BD28B81
@@
 	5050 2400 5400 2400
 $Comp
-L power:GND #PWR0109
-U 1 1 5BD28BC1
-P 5050 2900
-F 0 "#PWR0109" H 5050 2650 50  0001 C CNN
-F 1 "GND" H 5055 2727 50  0000 C CNN
-F 2 "" H 5050 2900 50  0001 C CNN
-F 3 "" H 5050 2900 50  0001 C CNN
-	1    5050 2900
-	1    0    0    -1
-$EndComp
-$Comp
 L power:GND #PWR0110
 U 1 1 5BD28BC7
-P 5700 2750
-F 0 "#PWR0110" H 5700 2500 50  0001 C CNN
-F 1 "GND" H 5705 2577 50  0000 C CNN
-F 2 "" H 5700 2750 50  0001 C CNN
-F 3 "" H 5700 2750 50  0001 C CNN
-	1    5700 2750
-	1    0    0    -1
-$EndComp
-Wire Wire Line
-	5700 2750 5700 2600
+P 5700 2850
+F 0 "#PWR0110" H 5700 2600 50  0001 C CNN
+F 1 "GND" H 5705 2677 50  0000 C CNN
+F 2 "" H 5700 2850 50  0001 C CNN
+F 3 "" H 5700 2850 50  0001 C CNN
+	1    5700 2850
+	1    0    0    -1
+$EndComp
 $Comp
 L Diode:LL4148 D3
@@
 	1    0    0    -1
 $EndComp
-Wire Wire Line
-	5050 2750 5050 2900
 $Comp
 L Device:R_Small R4
@@
 Text HLabel 5050 2400 0    50   Input ~ 0
 Out_1
-Text HLabel 5300 3550 0    50   Input ~ 0
+Text HLabel 5050 4500 0    50   Input ~ 0
 Out_2
 $Comp
@@
 Text Label 7150 3050 0    50   ~ 0
 K2_NC
+Text HLabel 5050 1200 0    50   Input ~ 0
+VCC_5V
+Wire Wire Line
+	5050 1200 5050 1450
+Wire Wire Line
+	5050 1450 5300 1450
+Connection ~ 5300 1450
+Text HLabel 4850 2850 0    50   Input ~ 0
+GND
+Wire Wire Line
+	4850 2850 5050 2850
+Wire Wire Line
+	5700 2600 5700 2850
+Connection ~ 5700 2850
+Wire Wire Line
+	5050 2750 5050 2850
+Connection ~ 5050 2850
+Wire Wire Line
+	5050 2850 5700 2850
+$Comp
+L power:GND #PWR0107
+U 1 1 5BE9AAA2
+P 5700 4900
+F 0 "#PWR0107" H 5700 4650 50  0001 C CNN
+F 1 "GND" H 5705 4727 50  0000 C CNN
+F 2 "" H 5700 4900 50  0001 C CNN
+F 3 "" H 5700 4900 50  0001 C CNN
+	1    5700 4900
+	1    0    0    -1
+$EndComp
+Wire Wire Line
+	5700 4900 5700 4700
 $EndSCHEMATC
